File: PCB/KiCAD/Zinnia2_0_5.kicad_pcb (KiCad board)
At the start: 2 copper layers, 125.4 x 90.3 mm, 115 parts, among them J1 Conn_01x06_Female, J11 Conn_01x02, J14 Conn_01x06, J15 Conn_01x06, J2 Conn_01x02, J4 Conn_01x01, J5 Rumble, J6 Conn_01x06, J9 USB_B_Micro, Q1 Q_NMOS_GSD, Q2 Q_PMOS_GDS, Q3 Q_NMOS_GSD, SW1 A, SW10 Dup, SW11 Dright, SW12 Ddown, SW2 B, SW3 X, SW4 Y, SW5 Start, SW6 L, SW7 R, SW8 Z, SW8L ZL, SW9 Dleft, U1 MCP3002, U10 DRV5055A2xDBZxQ1, U11 DRV5055A2xDBZxQ1, U2 Stickbox_Assembly_Main, U3 MCP3002, U4 DRV5055A2xDBZxQ1, U5 Stickbox_Assembly_CStick, U6 AMS1117-3.3, U7 W25Q128JVS, U8 RP2040, U9 DRV5055A2xDBZxQ1, Y1 Crystal_GND24

Commit message: MOUSEY THRU HOLE
U ALREADY KNOW
Parts:
- removed the REF** at (182.9, 40.8)
- removed the REF** at (188.2, 54.1)
- removed the REF** at (181.9, 63.8)
- SW1, SW3, SW4: footprint PhobGCC_2_0_0_footprints:ABXY_Contact_Omron_Switch -> PhobGCC_2_0_0_footprints:ABXY_Contact_Omron_Switch_b3F

Commit message: B3f pad test
Connections:
- SW1 pad : (no net) -> GND
- SW1 pad 5: GND -> /A
- SW2 pad : (no net) -> GND
- SW2 pad 5: GND -> /B
- SW3 pad : (no net) -> GND
- SW3 pad 5: GND -> /X
- SW4 pad : (no net) -> GND
- SW4 pad 5: GND -> /Y
Routing:
- net /B: track 39.2 -> 51.9 mm
- net GND: track 182.6 -> 171.0 mm
- net /X: track 61.2 -> 72.2 mm
- net /A: track 48.7 -> 56.6 mm
- net /Y: track 48.1 -> 54.3 mm
Other:
- board text added: "Zinnia 2.0.5"
- board text added: "github.com/plantsgcc/Zinnia2_0_5"
- board text removed: "PhloraGCC 2.0.2"
- board text removed: "github.com/plantsgcc/phloraGCC"

Commit message: Pad Updated
Parts:
- SW2: footprint PhobGCC_2_0_0_footprints:ABXY_Contact_Omron_Switch -> Library:ABXY_Contact_Omron_Switch_b3F_v2
- SW3, SW4: footprint PhobGCC_2_0_0_footprints:ABXY_Contact_Omron_Switch_b3F -> Library:ABXY_Contact_Omron_Switch_b3F_v2
Connections:
- SW1 pad : GND -> (no net)
- SW2 pad : GND -> (no net)
- SW3 pad : GND -> (no net)
- SW4 pad : GND -> (no net)
Routing:
- net /X: track 72.2 -> 65.4 mm, vias 0 -> 3
- net /B: track 51.9 -> 45.9 mm, vias 0 -> 3
- net /A: track 56.6 -> 54.6 mm, vias 0 -> 3
- net /Y: track 54.3 -> 53.9 mm, vias 0 -> 3
