File: PCB/KiCAD/Zinnia2_0_5.kicad_pcb (KiCad board)
At the start: 2 copper layers, 125.4 x 90.3 mm, 112 parts, among them J1 Conn_01x06_Female, J11 Conn_01x02, J14 Conn_01x06, J15 Conn_01x06, J2 Conn_01x02, J4 Conn_01x01, J5 Rumble, J6 PinSocket_1x04_P2.00mm_Vertic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, J9 USB_B_Micro, Q1 Q_NMOS_GSD, Q2 Q_PMOS_GDS, Q3 Q_NMOS_GSD, SW1 A, SW10 Dup, SW11 Dright, SW12 Ddown, SW2 B, SW3 X, SW4 Y, SW5 Start, SW6 L, SW7 R, SW8 Z, SW8L ZL, SW9 Dleft, U1 MCP3002, U10 DRV5055Z3QDBZT, U11 DRV5055Z3QDBZT, U12 USBLC6-2P6, U13 USBLC6-2P6, U2 Stickbox_Assembly_Main, U3 MCP3002, U4 DRV5055Z3QDBZT, U5 Stickbox_Assembly_CStick, U6 AMS1117-3.3, U7 W25Q128JVS, U8 RP2040, U9 DRV5055Z3QDBZT, Y1 Crystal_GND24

Commit message: New PC
Untested
Parts:
- added ?: , , F.Cu at (92.7, 69.1)
- RV1, RV2: footprint PhobGCC_2_0_0_footprints:GCC_Slider -> footprints:f
- SW1: footprint PhobGCC_2_0_0_footprints:ABXY_Contact_Omron_Switch_b3F -> footprints:ABXY_Contact_Omron_Switch_b3F_v2
- SW2, SW3, SW4: footprint Library:ABXY_Contact_Omron_Switch_b3F_v2 -> footprints:ABXY_Contact_Omron_Switch_b3F_v2
Connections:
- SW1 pad : GND -> (no net)
- SW2 pad : GND -> (no net)
- SW3 pad : GND -> (no net)
- SW4 pad : GND -> (no net)
Routing:
- net GND: track 162.6 -> 154.2 mm, vias 52 -> 54
- net +3V3: track 72.6 -> 77.6 mm, vias 16 -> 18
- net +5V: track 161.7 -> 160.9 mm
- net /A: track 46.9 -> 46.2 mm
- added copper zone on B.Cu, net +1V1
- added copper zone on B.Cu, net +3V3
- added copper zone on B.Cu, net +5V
- added copper zone on F.Cu, net +5V
- added copper zone on B.Cu, net /CLK
- added copper zone on F.Cu, net /CLK
- added copper zone on B.Cu, net /CS1
- added copper zone on F.Cu, net /CS1
- added copper zone on B.Cu, net /CS2
- added copper zone on F.Cu, net /CS2
- added copper zone on B.Cu, net /CS2_2
- added copper zone on F.Cu, net /CS2_2
- added copper zone on B.Cu, net /Din
- added copper zone on F.Cu, net /Din
- added copper zone on B.Cu, net /Dout
- added copper zone on F.Cu, net /Dout
- added copper zone on F.Cu, net /Dout2
- added copper zone on F.Cu, net /GCC_DATA
- added copper zone on F.Cu, net /GND_C
- added copper zone on F.Cu, net /GPIO13
- added copper zone on F.Cu, net /GPIO14
- added copper zone on F.Cu, net /GPIO15
- added copper zone on B.Cu, net /H1XS
- added copper zone on F.Cu, net /H1XS
- added copper zone on B.Cu, net /H1YS
- added copper zone on F.Cu, net /H1YS
- added copper zone on B.Cu, net /H2XS
- added copper zone on F.Cu, net /H2XS
- added copper zone on B.Cu, net /H2YS
- added copper zone on F.Cu, net /H2YS
- added copper zone on B.Cu, net /L
- added copper zone on F.Cu, net /L
- added copper zone on B.Cu, net /Ladder1
- added copper zone on F.Cu, net /Ladder1
- added copper zone on B.Cu, net /Ladder2
- added copper zone on F.Cu, net /Ladder2
- added copper zone on B.Cu, net /Ladder3
- added copper zone on F.Cu, net /Ladder3
- added copper zone on B.Cu, net /Ladder4
- added copper zone on F.Cu, net /Ladder4
- added copper zone on B.Cu, net /Lanalog
- added copper zone on F.Cu, net /Lanalog
- added copper zone on B.Cu, net /LeftZ
- added copper zone on F.Cu, net /LeftZ
- added copper zone on B.Cu, net /QSPI_SS
- added copper zone on F.Cu, net /QSPI_SS
- added copper zone on B.Cu, net /R
- added copper zone on F.Cu, net /R
- added copper zone on B.Cu, net /Ranalog
- added copper zone on F.Cu, net /Ranalog
- added copper zone on B.Cu, net /Rumble
- added copper zone on F.Cu, net /Rumble
- added copper zone on B.Cu, net /Start
- added copper zone on F.Cu, net /Start
- added copper zone on B.Cu, net /USB_D+
- added copper zone on F.Cu, net /USB_D+
- added copper zone on B.Cu, net /USB_D-
- added copper zone on F.Cu, net /USB_D-
- added copper zone on F.Cu, net /V
- added copper zone on F.Cu, net GND
- added copper zone on B.Cu, net Net-(D2-Pad2)
- added copper zone on F.Cu, net Net-(D2-Pad2)
- added copper zone on B.Cu, net Net-(J8-Pad6)
- added copper zone on F.Cu, net Net-(J8-Pad6)
- added copper zone on B.Cu, net VCC
